File: Eagle/RaspiLabBoard.brd (EAGLE design)
At the start: 65 x 56 mm, 18 parts

Commit message: Hardware version 2
As ordered from Aisler.net 20190519
Parts:
- removed SV2: (no value), con-lsta:FE07
- added C3, C5: (no value), rcl:E2-5
- added C6, C7: 100nF, SparkFun-Passives:0805
- added C8, C9: 22p, SparkFun-Passives:0805
- added J1, J2, J3: (no value), SparkFun-Connectors:1X02
- added Q1: 8MHz, special:QS
- added R2: 10k, SparkFun-Resistors:0805
- added R3: 120, SparkFun-Resistors:0805
- added U1: MCP2515, SparkFun-IC-Comms:SO18W
- added U2: MCP2551, SparkFun-IC-Comms:SO08
Connections:
- removed net 3V3: JP2.1, JP4.5, PH1.1, SV1.7, SV1.8
- removed net GND: C1.2, C2.2, C21.-, C4.2, D1.3, D2.3, D3.3, D8.4, D8.5, D8.6, JP2.25, JP2.30, JP2.34, JP2.6, JP2.9, JP4.4, S1.1, S2.1, SV1.5, SV1.6, SV2.2
- removed net GPIO14: C21.+, JP2.8, PH1.2
- new net CANH: J1.1, R3.1, U2.7
- new net CANL: J1.2, J3.2, U2.6
- new net GPIO12: C21.+, JP2.32, PH1.2
- new net N$10: J3.1, R3.2
- new net N$4: R2.1, U1.17
- new net N$7: C9.2, Q1.2, U1.8
- new net N$9: C8.2, Q1.1, U1.7
- new net RX: J2.1, JP2.10
- new net RXD: U1.2, U2.4
- new net TX: J2.2, JP2.8
- new net TXD: U1.1, U2.1
- new net VDD: C5.+, C7.1, JP2.1, JP4.5, PH1.1, R2.2, SV1.7, SV1.8, U1.18
- new net VSS: C1.2, C2.2, C21.-, C3.-, C4.2, C5.-, C6.1, C7.2, C8.1, C9.1, D1.3, D2.3, D3.3, D8.4, D8.5, D8.6, JP2.25, JP2.30, JP2.34, JP2.6, JP2.9, JP4.4, S1.1, S2.1, SV1.5, SV1.6, U1.9, U2.2, U2.8
- net 5V: now also C3.+, C6.2, U2.3; no longer SV2.1
- net CS: now also U1.16; no longer SV2.3
- net INT: now also U1.12; no longer SV2.7
- net SCK: now also U1.13; no longer SV2.6
- net SI: now also U1.14; no longer SV2.5
- net SO: now also U1.15; no longer SV2.4
Routing:
- net VSS: track 0.00 -> 277.7 mm, vias 0 -> 4
- net GND: track 226.7 -> 0.00 mm, vias 4 -> 0
- net GPIO12: track 0.00 -> 88.1 mm
- net VDD: track 0.00 -> 86.1 mm, vias 0 -> 1
- net 3V3: track 71.1 -> 0.00 mm
- net GPIO14: track 54.1 -> 0.00 mm
- net 5V: track 62.5 -> 97.9 mm
- net CANL: track 0.00 -> 25.3 mm
- net CANH: track 0.00 -> 20.4 mm
- net GPIO13: track 124.9 -> 105.3 mm
- net SDA: track 70.2 -> 51.6 mm
- net TX: track 0.00 -> 18.0 mm
- net CS: track 16.2 -> 34.1 mm
- net GPIO6: track 129.4 -> 147.3 mm
- net N$7: track 0.00 -> 17.6 mm
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- added copper zone on layer 1, net VSS
- added copper zone on layer 16, net VSS
- removed copper zone on layer 1, net GND
- removed copper zone on layer 16, net GND
Other:
- board text added: "3.3V!"
- board text added: "CANH"
- board text added: "CANL"
- board text added: "GP12"
- board text added: "RX"
- board text added: "RaspiLabBoard v. 2 Design: Pär Sundbäck github.com/teddycool"
- board text added: "TX"
- board text removed: "GP14"
- board text removed: "MCP2515 CAN module"
- board text removed: "RaspiLabBoard v. 1 Design: Pär Sundbäck github.com/teddycool"
- board text removed: "SPI: 1: 5V 2: GND 3: CS 4: SO 5: SI 6: SCK 7: INT"
