File: Eagle/RaspiLabBoard.sch (EAGLE design)
At the start: 18 parts

Commit message: Hardware version 2
As ordered from Aisler.net 20190519
Parts:
- removed SV2: (no value), con-lsta:FE07-1
- added C3, C5: (no value), rcl:CPOL-USE2-5
- added C6, C7: 100nF, SparkFun-Passives:CAP0805
- added C8, C9: 22p, SparkFun-Passives:CAP0805
- added J1, J2, J3: (no value), SparkFun-Connectors:CONN_02
- added Q1: 8MHz, special:XTAL/S
- added R2: 10k, SparkFun-Resistors:RESISTOR0805-RES
- added R3: 120, SparkFun-Resistors:RESISTOR0805-RES
- added U1: MCP2515, SparkFun-IC-Comms:MCP2515(MCP2510)SO
- added U2: MCP2551, SparkFun-IC-Comms:MCP2551
Connections:
- removed net 3V3: JP2.1, JP4.5, PH1.1, SV1.7, SV1.8
- removed net GND: C1.2, C2.2, C21.-, C4.2, D1.VSS, D2.VSS, D3.VSS, D8.BLU-C, D8.GRN-C, D8.RED-C, JP2.25, JP2.30, JP2.34, JP2.6, JP2.9, JP4.4, S1.1, S2.1, SV1.5, SV1.6, SV2.2
- removed net GPIO14: C21.+, JP2.8, PH1.2
- new net CANH: J1.1, R3.1, U2.CANH
- new net CANL: J1.2, J3.2, U2.CANL
- new net GPIO12: C21.+, JP2.32, PH1.2
- new net N$10: J3.1, R3.2
- new net N$4: R2.1, U1>NAME.RESET
- new net N$7: C9.2, Q1.2, U1>NAME.OSC1
- new net N$9: C8.2, Q1.1, U1>NAME.OSC2
- new net RX: J2.1, JP2.10
- new net RXD: U1>NAME.RXCAN, U2.RXD
- new net TX: J2.2, JP2.8
- new net TXD: U1>NAME.TXCAN, U2.TXD
- new net VDD: C5.+, C7.1, JP2.1, JP4.5, PH1.1, R2.2, SV1.7, SV1.8
- new net VSS: C1.2, C2.2, C21.-, C3.-, C4.2, C5.-, C6.1, C7.2, C8.1, C9.1, D1.VSS, D2.VSS, D3.VSS, D8.BLU-C, D8.GRN-C, D8.RED-C, JP2.25, JP2.30, JP2.34, JP2.6, JP2.9, JP4.4, S1.1, S2.1, SV1.5, SV1.6, U2.RS, U2.VSS
- net 5V: now also C3.+, C6.2, U2.VDD; no longer SV2.1
- net CS: now also U1>NAME.CS; no longer SV2.3
- net INT: now also U1>NAME.INT; no longer SV2.7
- net SCK: now also U1>NAME.SCK; no longer SV2.6
- net SI: now also U1>NAME.SI; no longer SV2.5
- net SO: now also U1>NAME.SO; no longer SV2.4
Other:
- note removed: "RPi Pin RPi Label CAN Module 02---------5V------------VCC 06---------GND-----------GND 19---------GPIO10--------MOSI (SI) 21---------GPIO9---------MISO (SO) 22---------GPIO25--------INT 23---------GPIO11--------SCK 24---------GPIO8---------CS"
- moved on the sheet: C1, C2, C21, C4, D1, D2, D3, D8, JP2, PH1, R1, R13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
